File: MoBaSbS-002-AnschaltGruppev3/MoBaSbS-002-AnschaltGruppev3.kicad_pcb (KiCad board)
At the start: 2 copper layers, 58.4 x 59.1 mm, 25 parts, among them J1 RJ45, J2 RJ45, J3 Conn_02x04_Top_Bottom, J4 Conn_02x04_Top_Bottom, P1 PSS254, P4 2x5_Buchse, P5 Wago, P6 Wago

Commit message: More work on that PCB, update to KiCad 9
Parts:
- added D3: WS2812B-2020, LED_SMD:LED_WS2812B-2020_PLCC4_2.0x2.0mm, F.Cu at (119.7, 155.5)
- added JP1: SolderJumper_2_Open, Jumper:SolderJumper-2_P1.3mm_Open_RoundedPad1.0x1.5mm, B.Cu at (186.6, 154.9)
- added JP2: SolderJumper_2_Open, Jumper:SolderJumper-2_P1.3mm_Open_RoundedPad1.0x1.5mm, B.Cu at (186.6, 151.4)
- F1, F2: footprint Fuse_Holders_and_Fuses:Fuseholder5x20_horiz_SemiClosed_Casing10x25mm -> Fuse:Fuseholder_Littelfuse_Nano2_154x
- J3: footprint Connector_PinSocket_2.54mm:PinSocket_2x04_P2.54mm_Horizontal -> Connector_PinSocket_2.54mm:PinSocket_2x05_P2.54mm_Horizontal
- J4: footprint Connector_PinHeader_2.54mm:PinHeader_2x04_P2.54mm_Horizontal -> Connector_PinHeader_2.54mm:PinHeader_2x05_P2.54mm_Horizontal
- P5, P6: footprint Molex MiniGit Jr 1x4:CONN_5566-04A_MOL -> Molex_MiniFitJr_1x4:CONN_5566-04A_MOL
- moved C2 26.7 mm to (116.9, 120.0), turned to 180 degrees
- moved C1 24.7 mm to (117.1, 130.8), turned to 180 degrees
- moved J3 22.4 mm to (143.7, 129.4)
- moved C4 22.0 mm to (114.3, 122.6), turned to 180 degrees
- moved C3 21.8 mm to (114.3, 133.3), turned to 180 degrees
- moved J4 17.3 mm to (143.7, 108.7)
- moved A1 16.1 mm to (137.3, 94.0)
- moved F1 14.1 mm to (148.8, 121.9)
- moved F2 9.71 mm to (148.8, 135.9)
- moved P6 4.87 mm to (127.6, 120.1)
Connections:
- J3 pad 1: Net-(J3-Pin_1) -> unconnected-(J3-Pin_1-Pad1)
- J3 pad 2: /5V -> Net-(D3-DIN)
- J3 pad 3: GND -> Net-(J3-Pin_3)
- J3 pad 4: Net-(J1-Pin_3) -> Net-(J3-Pin_4)
- J3 pad 5: Net-(J3-Pin_5) -> /5V
- J3 pad 8: Net-(J1-Pin_6) -> GND
- J4 pad 2: /5V -> unconnected-(J4-Pin_2-Pad2)
- J4 pad 3: GND -> unconnected-(J4-Pin_3-Pad3)
- J4 pad 5: unconnected-(J4-Pin_5-Pad5) -> /5V
- J4 pad 8: unconnected-(J4-Pin_8-Pad8) -> GND
- P4 pad 11: Net-(J3-Pin_1) -> Net-(J3-Pin_3)
- P4 pad 12: Net-(J3-Pin_5) -> Net-(J3-Pin_4)
Routing:
- net /12V PRE: track 68.9 -> 34.6 mm, vias 0 -> 1
- net +12V: track 90.1 -> 55.8 mm, vias 0 -> 1
- net /5V PRE: track 14.8 -> 31.6 mm, vias 0 -> 1
- net +5V: track 66.6 -> 50.5 mm
- net GND: track 152.2 -> 160.0 mm

Commit message: More work on the PCB
Parts:
- removed H5, H6: MountingHole_Pad, MountingHole:MountingHole_2.7mm_M2.5_DIN965_Pad
- removed J3: Conn_02x04_Top_Bottom, Connector_PinSocket_2.54mm:PinSocket_2x05_P2.54mm_Horizontal
- removed J4: Conn_02x04_Top_Bottom, Connector_PinHeader_2.54mm:PinHeader_2x05_P2.54mm_Horizontal
- R1, R2: moved to F.Cu
- moved JP2 62.0 mm to (124.7, 149.9)
- moved JP1 58.4 mm to (128.5, 149.9)
- moved R1 47.9 mm to (161.5, 120.0), turned to 90 degrees
- moved D1 46.2 mm to (164.1, 120.0), turned to 90 degrees
- moved D2 28.7 mm to (164.2, 127.6), turned to -90 degrees
- moved R2 26.5 mm to (161.5, 127.6), turned to -90 degrees
- moved C3 20.6 mm to (134.8, 131.4)
- moved H3 20.3 mm to (111.5, 80.6)
- moved H2 20.3 mm to (163.4, 80.6)
- moved C1 20.2 mm to (137.2, 131.4)
- moved C2 14.3 mm to (130.9, 122.6)
- moved C4 14.0 mm to (128.3, 122.6)
- moved P6 12.7 mm to (114.9, 119.9)
- moved P5 12.7 mm to (145.4, 120.0)
- moved F2 9.52 mm to (156.4, 130.2)
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Connections:
- A1 pad 40: /5V -> +5V
- D3 pad 3: Net-(D3-DIN) -> unconnected-(D3-DIN-Pad3)
- D3 pad 4: /5V -> +5V
Routing:
- net +5V: track 50.5 -> 85.5 mm
- net GND: track 160.0 -> 141.7 mm
- net /12V PRE: track 34.6 -> 48.1 mm, vias 1 -> 0
- net /5V PRE: track 31.6 -> 43.7 mm, vias 1 -> 0
- net Net-(J1-Pin_4): track 46.6 -> 37.6 mm
- net Net-(JP1-A): track 0.00 -> 7.78 mm, vias 0 -> 1
- net Net-(J1-Pin_5): track 44.0 -> 36.2 mm
- net Net-(JP2-A): track 0.00 -> 6.48 mm
- net Net-(D1-A): track 1.55 -> 3.91 mm, vias 1 -> 0
- net Net-(D2-A): track 1.65 -> 3.97 mm, vias 1 -> 0
- net +12V: track 55.8 -> 55.7 mm, vias 1 -> 0
Other:
- board size 58.4 x 59.1 mm -> 58.4 x 80 mm

Commit message: Added a few PCBs
Parts:
- added IC1: TJA1057BT, CAN Transceiver:SOIC127P600X175-8N, F.Cu at (140.9, 98.8)
- added IC2: SP3485EN-L_TR, RS485:SOIC127P600X175-8N, F.Cu at (115.8, 104.5)
- A1: footprint Module:RaspberryPi_Pico_Common_Unspecified -> Module_RaspberryPi_Pico:RaspberryPi_Pico_Original_SMD; moved to B.Cu
- moved C4 6.43 mm to (134.7, 122.4)
- moved C2 6.30 mm to (137.3, 122.4)
- moved A1 0.51 mm to (139.9, 100.2), turned to -90 degrees
Connections:
- A1 pad 36: unconnected-(A1-3V3-Pad36) -> /+3V3
Routing:
- net Net-(J1-Pin_6): track 0.00 -> 44.0 mm
- net Net-(J1-Pin_3): track 0.36 -> 41.4 mm
- net +5V: track 85.5 -> 116.2 mm, vias 0 -> 1
- net /+3V3: track 0.00 -> 11.3 mm, vias 0 -> 1
- net GND: track 141.7 -> 144.9 mm, vias 0 -> 1
Other:
- outline, holes or cut-outs redrawn

Commit message: Only some finishing touches left
Parts:
- added C5: 100nF, Capacitor_SMD:C_0603_1608Metric, F.Cu at (139.2, 101.9)
- added C6: 100nF, Capacitor_SMD:C_0603_1608Metric, F.Cu at (139.3, 140.5)
- added C7: 100nF, Capacitor_SMD:C_0603_1608Metric, F.Cu at (143.2, 112.1)
- added C8: 100nF, Capacitor_SMD:C_0603_1608Metric, F.Cu at (140.6, 122.4)
- added IC3: MCP2518FDT-E_SL, CAN Controller:SOIC127P600X175-14N, F.Cu at (143.7, 106.7)
- added J3: Conn_02x03_Odd_Even, Connector_PinSocket_2.54mm:PinSocket_2x03_P2.54mm_Horizontal, F.Cu at (153.9, 140.1)
- added J4: Conn_01x03, Connector_PinHeader_2.54mm:PinHeader_1x03_P2.54mm_Vertical, F.Cu at (163.4, 109.2)
- added J5: Conn_02x05_Counter_Clockwise, Connector_IDC:IDC-Header_2x05_P2.54mm_Vertical, F.Cu at (162.1, 127.0)
- added J6: Conn_01x04, Connector_Molex:Molex_KK-254_AE-6410-04A_1x04_P2.54mm_Vertical, F.Cu at (160.2, 93.3)
- added J7: Conn_01x04, Connector_Molex:Molex_KK-254_AE-6410-04A_1x04_P2.54mm_Vertical, F.Cu at (160.2, 104.8)
- added J8: Conn_01x03, Connector_PinHeader_2.54mm:PinHeader_1x03_P2.54mm_Vertical, F.Cu at (146.3, 135.1)
- A1: footprint Module_RaspberryPi_Pico:RaspberryPi_Pico_Original_SMD -> Module_RaspberryPi_Pico:RaspberryPi_Pico_Original_SMD_HandSolder
- moved D2 46.2 mm to (118.3, 133.5), turned to 180 degrees
- moved R2 43.3 mm to (118.3, 130.8), turned to 180 degrees
- moved F2 40.9 mm to (115.8, 125.7), turned to 0 degrees
- moved D1 40.4 mm to (126.0, 133.3), turned to 0 degrees
- moved IC2 38.3 mm to (134.8, 137.8), turned to -90 degrees
- moved R1 37.2 mm to (126.0, 130.8), turned to 0 degrees
- moved C3 33.3 mm to (115.7, 104.2), turned to 90 degrees
- moved P6 33.0 mm to (127.8, 89.5), turned to 0 degrees
- moved C1 32.9 mm to (115.7, 106.6), turned to 90 degrees
- moved F1 29.1 mm to (128.5, 125.7), turned to 180 degrees
- moved C4 20.9 mm to (124.7, 104.1), turned to 90 degrees
- moved C2 20.2 mm to (124.7, 106.6), turned to 90 degrees
- moved P5 18.5 mm to (127.7, 114.7), turned to 0 degrees
- moved IC1 18.2 mm to (143.1, 116.8), turned to -90 degrees
- moved H4 14.2 mm to (149.3, 139.4)
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Connections:
- A1 pad 1: unconnected-(A1-GPIO0-Pad1) -> /IO_11
- A1 pad 10: unconnected-(A1-GPIO7-Pad10) -> /CAN_SDI
- A1 pad 11: unconnected-(A1-GPIO8-Pad11) -> /GPIO22
- A1 pad 12: unconnected-(A1-GPIO9-Pad12) -> /GPIO21
- A1 pad 14: unconnected-(A1-GPIO10-Pad14) -> /GPIO20
- A1 pad 15: unconnected-(A1-GPIO11-Pad15) -> /GPIO19
- A1 pad 16: unconnected-(A1-GPIO12-Pad16) -> /GPIO18
- A1 pad 17: unconnected-(A1-GPIO13-Pad17) -> /GPIO17
- A1 pad 19: unconnected-(A1-GPIO14-Pad19) -> /GPIO16
- A1 pad 2: unconnected-(A1-GPIO1-Pad2) -> /IO_12
- A1 pad 20: unconnected-(A1-GPIO15-Pad20) -> /GPIO15
- A1 pad 21: unconnected-(A1-GPIO16-Pad21) -> /I2C_SDA
- A1 pad 22: unconnected-(A1-GPIO17-Pad22) -> /I2C_SCL
- A1 pad 24: unconnected-(A1-GPIO18-Pad24) -> /WS2812
- A1 pad 25: unconnected-(A1-GPIO19-Pad25) -> /MOBA_OUT
- A1 pad 26: unconnected-(A1-GPIO20-Pad26) -> /MOBA_WRITE
- A1 pad 27: unconnected-(A1-GPIO21-Pad27) -> /MOBA_IN
- A1 pad 29: unconnected-(A1-GPIO22-Pad29) -> /CAN_INT
- A1 pad 31: unconnected-(A1-GPIO26_ADC0-Pad31) -> /CAN_OSC
- A1 pad 32: unconnected-(A1-GPIO27_ADC1-Pad32) -> /CAN_INT0
- A1 pad 34: unconnected-(A1-GPIO28_ADC2-Pad34) -> /CAN_INT1
- A1 pad 4: unconnected-(A1-GPIO2-Pad4) -> /IO_21
- A1 pad 5: unconnected-(A1-GPIO3-Pad5) -> /IO_22
- A1 pad 6: unconnected-(A1-GPIO4-Pad6) -> /CAN_SDO
- A1 pad 7: unconnected-(A1-GPIO5-Pad7) -> /CAN_CS
- A1 pad 9: unconnected-(A1-GPIO6-Pad9) -> /CAN_SCK
- A1 pad D1: (no net) -> /SWDCLK
- A1 pad D2: (no net) -> GND
- A1 pad D3: (no net) -> /SWDIO
- D3 pad 3: unconnected-(D3-DIN-Pad3) -> /WS2812
- IC1 pad 1: unconnected-(IC1-TXD-Pad1) -> /CAN_TX
- IC1 pad 2: unconnected-(IC1-GND-Pad2) -> GND
- IC1 pad 3: unconnected-(IC1-VCC-Pad3) -> +5V
- IC1 pad 4: unconnected-(IC1-RXD-Pad4) -> /CAN_RX
- IC1 pad 5: unconnected-(IC1-VIO-Pad5) -> /+3V3
- IC1 pad 6: unconnected-(IC1-CANL-Pad6) -> /CAN_H
- IC1 pad 7: unconnected-(IC1-CANH-Pad7) -> /CAN_L
- IC2 pad 1: unconnected-(IC2-RO-Pad1) -> /MOBA_IN
- IC2 pad 2: unconnected-(IC2-~{RE}-Pad2) -> /MOBA_WRITE
- IC2 pad 3: unconnected-(IC2-DE-Pad3) -> /MOBA_WRITE
- IC2 pad 4: unconnected-(IC2-DI-Pad4) -> /MOBA_OUT
- J1 pad 3: Net-(J1-Pin_3) -> /CAN_L
- J1 pad 4: Net-(IC2-B) -> Net-(J1-Pin_4)
- J1 pad 5: Net-(IC2-A) -> Net-(J1-Pin_5)
- J1 pad 6: Net-(J1-Pin_6) -> /CAN_H
- J2 pad 3: Net-(J1-Pin_3) -> /CAN_L
- J2 pad 4: Net-(IC2-B) -> Net-(J1-Pin_4)
- J2 pad 5: Net-(IC2-A) -> Net-(J1-Pin_5)
- J2 pad 6: Net-(J1-Pin_6) -> /CAN_H
- JP1 pad 1: Net-(JP1-A) -> Net-(IC2-B)
- JP1 pad 2: Net-(IC2-B) -> Net-(J1-Pin_4)
- JP2 pad 1: Net-(JP2-A) -> Net-(IC2-A)
- JP2 pad 2: Net-(IC2-A) -> Net-(J1-Pin_5)
- P4 pad 1: Net-(J1-Pin_3) -> /I2C_SDA
- P4 pad 11: Net-(JP1-A) -> Net-(IC2-B)
- P4 pad 12: Net-(JP2-A) -> Net-(IC2-A)
- P4 pad 2: Net-(J1-Pin_6) -> /I2C_SCL
Routing:
- net +5V: track 116.2 -> 203.0 mm, vias 1 -> 3
- net GND: track 144.9 -> 201.3 mm, vias 1 -> 12
- net /CAN_L: track 0.00 -> 54.3 mm, vias 0 -> 1
- net /CAN_H: track 0.00 -> 49.5 mm, vias 0 -> 1
- net Net-(J1-Pin_6): track 44.0 -> 0.00 mm
- net /WS2812: track 0.00 -> 43.8 mm, vias 0 -> 3
- net /+3V3: track 11.3 -> 54.4 mm, vias 1 -> 3
- net Net-(J1-Pin_3): track 41.4 -> 0.00 mm
- net Net-(J1-Pin_4): track 0.00 -> 37.6 mm, vias 0 -> 1
- net Net-(J1-Pin_5): track 0.00 -> 36.2 mm
- net /MOBA_IN: track 0.00 -> 22.1 mm, vias 0 -> 1
- net /I2C_SCL: track 0.00 -> 21.7 mm
- net /MOBA_WRITE: track 0.00 -> 21.4 mm, vias 0 -> 1
- net /MOBA_OUT: track 0.00 -> 18.3 mm, vias 0 -> 1
- net /I2C_SDA: track 0.00 -> 17.9 mm
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- added copper zone on B.Cu, net GND
- added copper zone on F.Cu, net GND
Other:
- outline, holes or cut-outs redrawn
