File: MoBaSbS-002-AnschaltGruppev3/MoBaSbS-002-AnschaltGruppev3.kicad_sch (KiCad schematic)
At the start: 27 parts, among them J1 RJ45, J2 RJ45, J3 Conn_02x04_Top_Bottom, J4 Conn_02x04_Top_Bottom, P1 PSS254, P4 2x5_Buchse, P5 Wago, P6 Wago

Commit message: More work on that PCB, update to KiCad 9
Parts:
- added D3: WS2812B-2020, LED_SMD:LED_WS2812B-2020_PLCC4_2.0x2.0mm, symbol LED:WS2812B-2020
- F1, F2: footprint Fuse_Holders_and_Fuses:Fuseholder5x20_horiz_SemiClosed_Casing10x25mm -> Fuse:Fuseholder_Littelfuse_Nano2_154x
- J3: footprint Connector_PinSocket_2.54mm:PinSocket_2x04_P2.54mm_Horizontal -> Connector_PinSocket_2.54mm:PinSocket_2x05_P2.54mm_Horizontal; symbol Connector_Generic:Conn_02x04_Top_Bottom -> Connector_Generic:Conn_02x05_Odd_Even
- J4: footprint Connector_PinHeader_2.54mm:PinHeader_2x04_P2.54mm_Horizontal -> Connector_PinHeader_2.54mm:PinHeader_2x05_P2.54mm_Horizontal; symbol Connector_Generic:Conn_02x04_Top_Bottom -> Connector_Generic:Conn_02x05_Odd_Even
- JP1, JP2: footprint (none) -> Jumper:SolderJumper-2_P1.3mm_Open_RoundedPad1.0x1.5mm
- P5, P6: footprint Molex MiniGit Jr 1x4:CONN_5566-04A_MOL -> Molex_MiniFitJr_1x4:CONN_5566-04A_MOL
Connections:
- net 5V: now also J3.5 (Pin_5), J4.5 (Pin_5), D3.4 (VDD); no longer J3.2 (Pin_2), J4.2 (Pin_2)
- net GND: now also J3.8 (Pin_8), J4.8 (Pin_8), D3.2 (VSS); no longer J3.3 (Pin_3), J4.3 (Pin_3)
- net at J1.3 (Pin_3), J2.3 (Pin_3), P4.1 (Pin_1): now also J3.9 (Pin_9); no longer J3.4 (Pin_4)
- net at J1.6 (Pin_6), J2.6 (Pin_6), P4.2 (Pin_2): now also J3.10 (Pin_10); no longer J3.8 (Pin_8)
- net at JP1.1 (A), P4.11 (Pin_11): now also J3.3 (Pin_3); no longer J3.1 (Pin_1)
- net at JP2.1 (A), P4.12 (Pin_12): now also J3.4 (Pin_4); no longer J3.5 (Pin_5)
- new net: D3.3 (DIN), J3.2 (Pin_2)
- no-connect marks 20 -> 23

Commit message: More work on the PCB
Parts:
- removed H5, H6: MountingHole_Pad, MountingHole:MountingHole_2.7mm_M2.5_DIN965_Pad, symbol Mechanical:MountingHole_Pad
- removed J3: Conn_02x04_Top_Bottom, Connector_PinSocket_2.54mm:PinSocket_2x05_P2.54mm_Horizontal, symbol Connector_Generic:Conn_02x05_Odd_Even
- removed J4: Conn_02x04_Top_Bottom, Connector_PinHeader_2.54mm:PinHeader_2x05_P2.54mm_Horizontal, symbol Connector_Generic:Conn_02x05_Odd_Even
Connections:
- net 5V is gone; now on net +5V: A1.40 (VBUS), D3.4 (VDD)
- no-connect marks 23 -> 19
Other:
- moved on the sheet: D3

Commit message: Added a few PCBs
Parts:
- added IC1: TJA1057BT, CAN Transceiver:SOIC127P600X175-8N, symbol TJA1057BT:TJA1057BT
- added IC2: SP3485EN-L_TR, RS485:SOIC127P600X175-8N, symbol SP3485EN-L_TR:SP3485EN-L_TR
- added IC3: MCP2518FDT-E_SL, SOIC127P600X175-14N, symbol MCP2518FDT-E_SL:MCP2518FDT-E_SL
- A1: footprint Module:RaspberryPi_Pico_Common_Unspecified -> Module_RaspberryPi_Pico:RaspberryPi_Pico_Original_SMD
Connections:
- net GND: now also IC2.5 (GND)
- net at J1.4 (Pin_4), J2.4 (Pin_4), JP1.2 (B): now also IC2.7 (B)
- net at J1.5 (Pin_5), J2.5 (Pin_5), JP2.2 (B): now also IC2.6 (A)
- net +3V3: now reaches A1.36 (3V3)
- net +3V3: now also IC2.8 (VCC)
- no-connect marks 19 -> 18

Commit message: Only some finishing touches left
Parts:
- added C5, C6, C7, C8: 100nF, Capacitor_SMD:C_0603_1608Metric, symbol Device:C
- added J3: Conn_02x03_Odd_Even, Connector_PinSocket_2.54mm:PinSocket_2x03_P2.54mm_Horizontal, symbol Connector_Generic:Conn_02x03_Odd_Even
- added J4, J8: Conn_01x03, Connector_PinHeader_2.54mm:PinHeader_1x03_P2.54mm_Vertical, symbol Connector_Generic:Conn_01x03
- added J5: Conn_02x05_Counter_Clockwise, Connector_IDC:IDC-Header_2x05_P2.54mm_Vertical, symbol Connector_Generic:Conn_02x05_Counter_Clockwise
- added J6, J7: Conn_01x04, Connector_Molex:Molex_KK-254_AE-6410-04A_1x04_P2.54mm_Vertical, symbol Connector_Generic:Conn_01x04
- A1: footprint Module_RaspberryPi_Pico:RaspberryPi_Pico_Original_SMD -> Module_RaspberryPi_Pico:RaspberryPi_Pico_Original_SMD_HandSolder; symbol RPi Pico:RaspberryPi_Pico -> MCU_Module_RaspberryPi_Pico:RaspberryPi_Pico_DebugPins
Connections:
- net +3V3: now also IC1.5 (VIO), IC3.14 (VDD), C5.2, C6.1, C8.2
- net +5V: now also IC1.3 (VCC), C7.1, J3.3 (Pin_3), J3.4 (Pin_4), J4.3 (Pin_3), J6.4 (Pin_4), J7.4 (Pin_4)
- net GND: now also A1.D2 (GND), IC1.2 (GND), IC3.7 (VSS), C5.1, C6.2, C7.2, C8.1, J3.5 (Pin_5), J3.6 (Pin_6), J5.1 (Pin_1), J6.1 (Pin_1), J7.1 (Pin_1), J8.2 (Pin_2)
- net CAN_L: now reaches J1.3 (Pin_3), J2.3 (Pin_3)
- net CAN_L: now also IC1.7 (CANH), J3.2 (Pin_2); no longer P4.1 (Pin_1)
- net at J1.4 (Pin_4), J2.4 (Pin_4), JP1.2 (B): no longer IC2.7 (B)
- net at J1.5 (Pin_5), J2.5 (Pin_5), JP2.2 (B): no longer IC2.6 (A)
- net CAN_H: now reaches J1.6 (Pin_6), J2.6 (Pin_6)
- net CAN_H: now also IC1.6 (CANL), J3.1 (Pin_1); no longer P4.2 (Pin_2)
- net at JP1.1 (A), P4.11 (Pin_11): now also IC2.7 (B)
- net at JP2.1 (A), P4.12 (Pin_12): now also IC2.6 (A)
- net CAN_TX: now reaches IC1.1 (TXD)
- net CAN_TX: now also IC3.1 (TXCAN)
- net CAN_RX: now reaches IC1.4 (RXD)
- net CAN_RX: now also IC3.2 (RXCAN)
- net MOBA_IN: now reaches IC2.1 (RO)
- net MOBA_IN: now also A1.27 (GPIO21)
- net MOBA_WRITE: now reaches IC2.2 (~{RE})
- net MOBA_WRITE: now also A1.26 (GPIO20), IC2.3 (DE)
- net MOBA_OUT: now reaches IC2.4 (DI)
- net MOBA_OUT: now also A1.25 (GPIO19)
- net IO_11: now reaches A1.1 (GPIO0)
- net IO_11: now also J6.3 (Pin_3)
- net CAN_SDI: now reaches A1.10 (GPIO7)
- net CAN_SDI: now also IC3.11 (SDI)
- net GPIO22: now reaches A1.11 (GPIO8)
- net GPIO22: now also J5.9 (Pin_9)
- net GPIO21: now reaches A1.12 (GPIO9)
- net GPIO21: now also J5.8 (Pin_8)
- net GPIO20: now reaches A1.14 (GPIO10)
- net GPIO20: now also J5.7 (Pin_7)
- net GPIO19: now reaches A1.15 (GPIO11)
- net GPIO19: now also J5.6 (Pin_6)
- net GPIO18: now reaches A1.16 (GPIO12)
- net GPIO18: now also J5.5 (Pin_5)
- net GPIO17: now reaches A1.17 (GPIO13)
- net GPIO17: now also J5.4 (Pin_4)
- net GPIO16: now reaches A1.19 (GPIO14)
- net GPIO16: now also J5.3 (Pin_3)
- net IO_12: now reaches A1.2 (GPIO1)
- net IO_12: now also J6.2 (Pin_2)
- net GPIO15: now reaches A1.20 (GPIO15)
- net GPIO15: now also J5.2 (Pin_2)
- net I2C_SDA: now reaches A1.21 (GPIO16)
- net I2C_SDA: now also P4.1 (Pin_1)
- net I2C_SCL: now reaches A1.22 (GPIO17)
- net I2C_SCL: now also P4.2 (Pin_2)
- net WS2812: now reaches A1.24 (GPIO18)
- net WS2812: now also D3.3 (DIN)
- net CAN_INT: now reaches A1.29 (GPIO22)
- net CAN_INT: now also IC3.4 (~{INT})
- net CAN_OSC: now reaches A1.31 (GPIO26_ADC0)
- net CAN_OSC: now also IC3.6 (OSC1)
- net CAN_INT0: now reaches A1.32 (GPIO27_ADC1)
- net CAN_INT0: now also IC3.9 (~{INT0}/GPIO0/XSTBY)
- net CAN_INT1: now reaches A1.34 (GPIO28_ADC2)
- net CAN_INT1: now also IC3.8 (~{INT1}/GPIO1)
- net IO_21: now reaches A1.4 (GPIO2)
- net IO_21: now also J7.3 (Pin_3)
- net IO_22: now reaches A1.5 (GPIO3)
- net IO_22: now also J7.2 (Pin_2)
- net CAN_SDO: now reaches A1.6 (GPIO4)
- net CAN_SDO: now also IC3.12 (SDO)
- net CAN_CS: now reaches A1.7 (GPIO5)
- net CAN_CS: now also IC3.13 (NCS)
- net CAN_SCK: now reaches A1.9 (GPIO6)
- net CAN_SCK: now also IC3.10 (SCK)
- new net: J4.2 (Pin_2), J5.10 (Pin_10)
- new net 3V3: J4.1 (Pin_1)
- new net SWDCLK: A1.D1 (SWCLK), J8.1 (Pin_1)
- new net SWDIO: A1.D3 (SWDIO), J8.3 (Pin_3)
- no-connect marks 18 -> 20
Other:
- note added: "Extra 3v3 Input einbauen und 3v3 vom RP2040 trennbar machen, falls es nicht ausreicht Pin am CAN-Transceiver verbinden 2020 - Footprint prüfen"
- moved on the sheet: D3, IC1, IC3

Commit message: Some more work
Connections:
- net +5V: now also A1.39 (VSYS); no longer A1.40 (VBUS)
- no-connect marks 20 -> 19
Changed lines of the file:
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@@
 		(at 132.08 49.53)
 	)
-	(no_connect
-		(at 238.76 59.69)
-	)
 	(wire
 		(pts
@@
 	(wire
 		(pts
+			(xy 238.76 57.15) (xy 238.76 59.69)
+		)
+		(stroke
+			(width 0)
+			(type default)
+		)
+	)
+	(wire
+		(pts
 			(xy 36.83 49.53) (xy 38.1 49.53)
 		)
@@
 		(pts
 			(xy 31.75 59.69) (xy 38.1 59.69)
-		)
-		(stroke
-			(width 0)
-			(type default)
-		)
-	)
-	(wire
-		(pts
-			(xy 243.84 57.15) (xy 243.84 59.69)
 		)
 		(stroke
@@
 		)
 	)
+	(label "+5V"
+		(at 238.76 57.15 90)
+		(effects
+			(font
+				(size 1.524 1.524)
+			)
+			(justify left bottom)
+		)
+	)
 	(label "GPIO17"
 		(at 120.65 180.34 180)
@@
 		)
 	)
-	(label "+5V"
-		(at 243.84 57.15 90)
-		(effects
-			(font
-				(size 1.524 1.524)
-			)
-			(justify left bottom)
-		)
-	)
