File: MoBaSbS-504-STM32Rueckmelder/MoBaSbS-504-STM32Rueckmelder.kicad_sch (KiCad schematic)
At the start: 15 parts, among them IC1 TJA1057BT, J1 RJ45, J2 RJ45, J3 Conn_02x05_Counter_Clockwise, J4 Conn_01x03, J5 Conn_02x05_Counter_Clockwise, J6 Conn_01x03, P1 PSS254

Commit message: Only some finishing touches left
Parts:
- added J7: Conn_02x03_Odd_Even, Connector_PinHeader_2.54mm:PinHeader_2x03_P2.54mm_Horizontal, symbol Connector_Generic:Conn_02x03_Odd_Even
Connections:
- net +5V: now also J7.3 (Pin_3), J7.4 (Pin_4)
- net GND: now also J7.5 (Pin_5), J7.6 (Pin_6)
- net at IC1.6 (CANL), J1.3 (Pin_3), J2.3 (Pin_3): now also J7.2 (Pin_2)
- net at IC1.7 (CANH), J1.6 (Pin_6), J2.6 (Pin_6): now also J7.1 (Pin_1)
Other:
- note added: "MoBaSbS Signal an RJ45 verbinden"
Changed lines of the file:
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@@
 	(generator_version "9.0")
 	(paper "A4")
+	(text "MoBaSbS Signal an RJ45 verbinden"
+		(exclude_from_sim no)
+		(at 135.382 25.654 0)
+		(effects
+			(font
+				(size 0.762 0.762)
+			)
+		)
+	)
 	(junction
 		(at 171.45 118.11)
@@
 	)
 	(junction
+		(at 171.45 132.08)
+		(diameter 0)
+		(color 0 0 0 0)
+	)
+	(junction
+		(at 147.32 129.54)
+		(diameter 0)
+		(color 0 0 0 0)
+	)
+	(junction
 		(at 173.99 125.73)
 		(diameter 0)
@@
 	(wire
 		(pts
+			(xy 165.1 152.4) (xy 166.37 152.4)
+		)
+		(stroke
+			(width 0)
+			(type default)
+		)
+	)
+	(wire
+		(pts
+			(xy 151.13 149.86) (xy 152.4 149.86)
+		)
+		(stroke
+			(width 0)
+			(type default)
+		)
+	)
+	(wire
+		(pts
 			(xy 25.4 67.31) (xy 26.67 67.31)
 		)
@@
 	(wire
 		(pts
+			(xy 147.32 147.32) (xy 147.32 129.54)
+		)
+		(stroke
+			(width 0)
+			(type default)
+		)
+	)
+	(wire
+		(pts
 			(xy 92.71 102.87) (xy 93.98 102.87)
 		)
@@
 	(wire
 		(pts
+			(xy 151.13 152.4) (xy 152.4 152.4)
+		)
+		(stroke
+			(width 0)
+			(type default)
+		)
+	)
+	(wire
+		(pts
+			(xy 165.1 149.86) (xy 166.37 149.86)
+		)
+		(stroke
+			(width 0)
+			(type default)
+		)
+	)
+	(wire
+		(pts
 			(xy 25.4 104.14) (xy 26.67 104.14)
 		)
@@
 	(wire
 		(pts
+			(xy 152.4 147.32) (xy 147.32 147.32)
+		)
+		(stroke
+			(width 0)
+			(type default)
+		)
+	)
+	(wire
+		(pts
 			(xy 39.37 106.68) (xy 40.64 106.68)
 		)
@@
 	(wire
 		(pts
-			(xy 119.38 129.54) (xy 173.99 129.54)
+			(xy 119.38 129.54) (xy 147.32 129.54)
 		)
 		(stroke
@@
 	(wire
 		(pts
+			(xy 165.1 147.32) (xy 171.45 147.32)
+		)
+		(stroke
+			(width 0)
+			(type default)
+		)
+	)
+	(wire
+		(pts
+			(xy 171.45 147.32) (xy 171.45 132.08)
+		)
+		(stroke
+			(width 0)
+			(type default)
+		)
+	)
+	(wire
+		(pts
 			(xy 114.3 102.87) (xy 115.57 102.87)
 		)
@@
 		(pts
 			(xy 39.37 101.6) (xy 40.64 101.6)
+		)
+		(stroke
+			(width 0)
+			(type default)
+		)
+	)
+	(wire
+		(pts
+			(xy 147.32 129.54) (xy 173.99 129.54)
 		)
 		(stroke
@@
 		)
 	)
+	(label "+5V"
+		(at 151.13 149.86 180)
+		(effects
+			(font
+				(size 1.27 1.27)
+			)
+			(justify right bottom)
+		)
+	)
 	(label "3V3"
 		(at 57.15 54.61 180)
@@
 		)
 	)
+	(label "+5V"
+		(at 166.37 149.86 0)
+		(effects
+			(font
+				(size 1.27 1.27)
+			)
+			(justify left bottom)
+		)
+	)
 	(label "GND"
 		(at 115.57 85.09 0)
@@
 		)
 	)
+	(label "GND"
+		(at 166.37 152.4 0)
+		(effects
+			(font
+				(size 1.27 1.27)
+			)
+			(justify left bottom)
+		)
+	)
 	(label "ADC1_IN15"
 		(at 25.4 104.14 180)
@@
 			)
 			(justify left bottom)
+		)
+	)
+	(label "GND"
+		(at 151.13 152.4 180)
+		(effects
+			(font
+				(size 1.27 1.27)
+			)
+			(justify right bottom)
 		)
 	)
@@
 					(unit 1)
 				)
+			)
+		)
+	)
+	(symbol
+		(lib_id "Connector_Generic:Conn_02x03_Odd_Even")
+		(at 157.48 149.86 0)
+		(unit 1)
+		(exclude_from_sim no)
+		(in_bom yes)
+		(on_board yes)
+		(dnp no)
+		(fields_autoplaced yes)
+		(property "Reference" "J7"
+			(at 158.75 140.97 0)
+			(effects
+				(font
+					(size 1.27 1.27)
+				)
+			)
+		)
+		(property "Value" "Conn_02x03_Odd_Even"
+			(at 158.75 143.51 0)
+			(effects
+				(font
+					(size 1.27 1.27)
+				)
+			)
+		)
+		(property "Footprint" "Connector_PinHeader_2.54mm:PinHeader_2x03_P2.54mm_Horizontal"
+			(at 157.48 149.86 0)
+			(effects
+				(font
+					(size 1.27 1.27)
+				)
+				(hide yes)
+			)
+		)
+		(property "Datasheet" "~"
+			(at 157.48 149.86 0)
+			(effects
+				(font
+					(size 1.27 1.27)
+				)
+				(hide yes)
+			)
+		)
+		(property "Description" "Generic connector, double row, 02x03, odd/even pin numbering scheme (row 1 odd numbers, row 2 even numbers), script generated (kicad-library-utils/schlib/autogen/connector/)"
+			(at 157.48 149.86 0)
+			(effects
+				(font
+					(size 1.27 1.27)
+				)
+				(hide yes)
+			)
+		)
+		(pin "6"
+		)
+		(pin "3"
+		)
+		(pin "5"
+		)
+		(pin "1"
+		)
+		(pin "2"
+		)
+		(pin "4"
+		)
+		(instances
+			(project ""
+				(path "/f189e98a-821f-4c13-81c8-99e5bf8af46f"
+					(reference "J7")
+					(unit 1)
+				)

Commit message: Some more work
Connections:
- net at J1.4 (Pin_4): now also J2.4 (Pin_4)
- net at J1.5 (Pin_5): now also J2.5 (Pin_5)
- no-connect marks 37 -> 33
Other:
- note removed: "MoBaSbS Signal an RJ45 verbinden"
Changed lines of the file:
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@@
 	(generator_version "9.0")
 	(paper "A4")
-	(text "MoBaSbS Signal an RJ45 verbinden"
-		(exclude_from_sim no)
-		(at 135.382 25.654 0)
-		(effects
-			(font
-				(size 0.762 0.762)
-			)
-		)
-	)
 	(junction
 		(at 171.45 118.11)
@@
 	)
 	(no_connect
-		(at 179.07 123.19)
-	)
-	(no_connect
 		(at 93.98 74.93)
 	)
@@
 	)
 	(no_connect
-		(at 179.07 88.9)
-	)
-	(no_connect
 		(at 93.98 59.69)
 	)
@@
 	)
 	(no_connect
-		(at 179.07 91.44)
-	)
-	(no_connect
 		(at 114.3 67.31)
 	)
@@
 	)
 	(no_connect
-		(at 179.07 120.65)
-	)
-	(no_connect
 		(at 179.07 130.81)
 	)
@@
 	(wire
 		(pts
+			(xy 166.37 123.19) (xy 166.37 91.44)
+		)
+		(stroke
+			(width 0)
+			(type default)
+		)
+	)
+	(wire
+		(pts
 			(xy 39.37 67.31) (xy 40.64 67.31)
 		)
@@
 	(wire
 		(pts
+			(xy 179.07 88.9) (xy 168.91 88.9)
+		)
+		(stroke
+			(width 0)
+			(type default)
+		)
+	)
+	(wire
+		(pts
 			(xy 69.85 132.08) (xy 72.39 132.08)
 		)
@@
 	(wire
 		(pts
+			(xy 168.91 120.65) (xy 179.07 120.65)
+		)
+		(stroke
+			(width 0)
+			(type default)
+		)
+	)
+	(wire
+		(pts
 			(xy 39.37 57.15) (xy 57.15 57.15)
 		)
@@
 	(wire
 		(pts
+			(xy 179.07 123.19) (xy 166.37 123.19)
+		)
+		(stroke
+			(width 0)
+			(type default)
+		)
+	)
+	(wire
+		(pts
 			(xy 39.37 106.68) (xy 40.64 106.68)
 		)
@@
 	(wire
 		(pts
+			(xy 166.37 91.44) (xy 179.07 91.44)
+		)
+		(stroke
+			(width 0)
+			(type default)
+		)
+	)
+	(wire
+		(pts
 			(xy 119.38 129.54) (xy 147.32 129.54)
 		)
@@
 		)
 		(stroke
+			(width 0)
+			(type default)
+		)
+	)
+	(wire
+		(pts
+			(xy 168.91 88.9) (xy 168.91 120.65)
+		)
+		(stroke
