File: MA-003-Pico/MA-003-Pico.kicad_sch (KiCad schematic)
At the start: 5 parts, among them M1 rs485_ttl_module, M2 rs485_ttl_module, M3 rs485_ttl_module, M4 rs485_ttl_module

Commit message: Some more work
Parts:
- removed M1, M2, M3, M4: rs485_ttl_module, RS485ToTTL:rs485_ttl_module, symbol RS485ToTTL:rs485_ttl_module
- added H1, H2, H3, H4: MountingHole_Pad, MountingHole:MountingHole_2.7mm_M2.5_DIN965_Pad, symbol Mechanical:MountingHole_Pad
- added J1: Power, Connector_Molex:Molex_KK-254_AE-6410-03A_1x03_P2.54mm_Vertical, symbol Connector_Generic:Conn_01x03
- added J2: I2C, Connector_Molex:Molex_KK-254_AE-6410-04A_1x04_P2.54mm_Vertical, symbol Connector_Generic:Conn_01x04
- added J3: Interface_A, Connector_IDC:IDC-Header_2x05_P2.54mm_Vertical, symbol Connector_Generic:Conn_02x05_Counter_Clockwise
- added J4: Interface_B, Connector_IDC:IDC-Header_2x05_P2.54mm_Vertical, symbol Connector_Generic:Conn_02x05_Counter_Clockwise
- added J5: Power_IB, Connector_PinHeader_2.54mm:PinHeader_1x03_P2.54mm_Vertical, symbol Connector_Generic:Conn_01x03
- added J6: Power_IA, Connector_PinHeader_2.54mm:PinHeader_1x03_P2.54mm_Vertical, symbol Connector_Generic:Conn_01x03
- added J7: Pico_On/Off, Connector_PinHeader_2.54mm:PinHeader_1x02_P2.54mm_Vertical, symbol Connector_Generic:Conn_01x02
- added J8: WS2812, Connector_Molex:Molex_KK-254_AE-6410-03A_1x03_P2.54mm_Vertical, symbol Connector_Generic:Conn_01x03
Connections:
- net GPIO_1: now reaches A1.1 (GPIO0)
- net GPIO_1: now also J3.2 (Pin_2)
- net GPIO_8: now reaches A1.10 (GPIO7)
- net GPIO_8: now also J3.9 (Pin_9)
- net GPIO_9: now reaches A1.11 (GPIO8)
- net GPIO_9: now also J4.2 (Pin_2)
- net GPIO_10: now reaches A1.12 (GPIO9)
- net GPIO_10: now also J4.3 (Pin_3)
- net GND: now reaches A1.13 (GND), A1.18 (GND), A1.23 (GND), A1.28 (GND), A1.3 (GND), A1.38 (GND), A1.8 (GND)
- net GND: now also A1.33 (AGND), J1.1 (Pin_1), J2.1 (Pin_1), J3.1 (Pin_1), J4.1 (Pin_1), J7.2 (Pin_2), J8.1 (Pin_1)
- net GPIO_11: now reaches A1.14 (GPIO10)
- net GPIO_11: now also J4.4 (Pin_4)
- net GPIO_12: now reaches A1.15 (GPIO11)
- net GPIO_12: now also J4.5 (Pin_5)
- net GPIO_13: now reaches A1.16 (GPIO12)
- net GPIO_13: now also J4.6 (Pin_6)
- net GPIO_14: now reaches A1.17 (GPIO13)
- net GPIO_14: now also J4.7 (Pin_7)
- net GPIO_15: now reaches A1.19 (GPIO14)
- net GPIO_15: now also J4.8 (Pin_8)
- net GPIO_2: now reaches A1.2 (GPIO1)
- net GPIO_2: now also J3.3 (Pin_3)
- net GPIO_16: now reaches A1.20 (GPIO15)
- net GPIO_16: now also J4.9 (Pin_9)
- net at A1.30 (RUN): now also J7.1 (Pin_1)
- net I2C_SDA: now reaches A1.31 (GPIO26_ADC0)
- net I2C_SDA: now also J2.2 (Pin_2)
- net I2C_SCL: now reaches A1.32 (GPIO27_ADC1)
- net I2C_SCL: now also J2.3 (Pin_3)
- net at A1.34 (GPIO28_ADC2): now also J8.2 (Pin_2)
- net 5V: now reaches A1.39 (VSYS)
- net 5V: now also J1.3 (Pin_3), J2.4 (Pin_4), J5.3 (Pin_3), J6.3 (Pin_3), J8.3 (Pin_3)
- net GPIO_3: now reaches A1.4 (GPIO2)
- net GPIO_3: now also J3.4 (Pin_4)
- net GPIO_4: now reaches A1.5 (GPIO3)
- net GPIO_4: now also J3.5 (Pin_5)
- net GPIO_5: now reaches A1.6 (GPIO4)
- net GPIO_5: now also J3.6 (Pin_6)
- net GPIO_6: now reaches A1.7 (GPIO5)
- net GPIO_6: now also J3.7 (Pin_7)
- net GPIO_7: now reaches A1.9 (GPIO6)
- net GPIO_7: now also J3.8 (Pin_8)
- new net: J4.10 (Pin_10), J5.2 (Pin_2)
- new net: J3.10 (Pin_10), J6.2 (Pin_2)
- new net 3V3: J1.2 (Pin_2), J5.1 (Pin_1), J6.1 (Pin_1)
- no-connect marks 0 -> 15

Commit message: Finishing the dmx ethernet pico
Connections:
- net GPIO_10: now also J4.8 (Pin_8); no longer J4.3 (Pin_3)
- net GPIO_11: now also J4.7 (Pin_7); no longer J4.4 (Pin_4)
- net GPIO_12: now also J4.6 (Pin_6); no longer J4.5 (Pin_5)
- net GPIO_13: now also J4.5 (Pin_5); no longer J4.6 (Pin_6)
- net GPIO_14: now also J4.4 (Pin_4); no longer J4.7 (Pin_7)
- net GPIO_15: now also J4.3 (Pin_3); no longer J4.8 (Pin_8)
- net GPIO_16: now also J4.2 (Pin_2); no longer J4.9 (Pin_9)
- net GPIO_9: now also J4.9 (Pin_9); no longer J4.2 (Pin_2)
Changed lines of the file:
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@@
+		)
+	)
+	(label "GPIO_14"
+		(at 204.47 129.54 180)
+		(effects
+			(font
+				(size 1.27 1.27)
+			)
+			(justify right bottom)
 		)
 	)
@@
 		)
 	)
-	(label "GPIO_16"
-		(at 219.71 124.46 0)
-		(effects
-			(font
-				(size 1.27 1.27)
-			)
-			(justify left bottom)
-		)
-	)
 	(label "GND"
 		(at 204.47 93.98 180)
@@
 		)
 	)
-	(label "GPIO_12"
-		(at 204.47 132.08 180)
-		(effects
-			(font
-				(size 1.27 1.27)
-			)
-			(justify right bottom)
-		)
-	)
 	(label "GND"
 		(at 102.87 114.3 0)
@@
 		)
 	)
+	(label "GPIO_15"
+		(at 204.47 127 180)
+		(effects
+			(font
+				(size 1.27 1.27)
+			)
+			(justify right bottom)
+		)
+	)
 	(label "5V"
 		(at 181.61 46.99 180)
@@
 		)
 	)
-	(label "GPIO_11"
-		(at 204.47 129.54 180)
-		(effects
-			(font
-				(size 1.27 1.27)
-			)
-			(justify right bottom)
-		)
-	)
 	(label "GND"
 		(at 189.23 109.22 180)
@@
 		)
 	)
-	(label "GPIO_14"
-		(at 219.71 129.54 0)
-		(effects
-			(font
-				(size 1.27 1.27)
-			)
-			(justify left bottom)
-		)
-	)
-	(label "GPIO_13"
-		(at 219.71 132.08 0)
-		(effects
-			(font
-				(size 1.27 1.27)
-			)
-			(justify left bottom)
+	(label "GPIO_16"
+		(at 204.47 124.46 180)
+		(effects
+			(font
+				(size 1.27 1.27)
+			)
+			(justify right bottom)
 		)
 	)
@@
 		)
 	)
+	(label "GPIO_10"
+		(at 219.71 127 0)
+		(effects
+			(font
+				(size 1.27 1.27)
+			)
+			(justify left bottom)
+		)
+	)
 	(label "GPIO_12"
 		(at 121.92 101.6 180)
@@
 		)
 	)
+	(label "GPIO_9"
+		(at 219.71 124.46 0)
+		(effects
+			(font
+				(size 1.27 1.27)
+			)
+			(justify left bottom)
+		)
+	)
 	(label "5V"
 		(at 240.03 124.46 180)
@@
 		)
 	)
-	(label "GPIO_15"
-		(at 219.71 127 0)
-		(effects
-			(font
-				(size 1.27 1.27)
-			)
-			(justify left bottom)
-		)
-	)
-	(label "GPIO_10"
-		(at 204.47 127 180)
-		(effects
-			(font
-				(size 1.27 1.27)
-			)
-			(justify right bottom)
-		)
-	)
 	(label "GPIO_5"
 		(at 121.92 83.82 180)
@@
 		)
 	)
+	(label "GPIO_11"
+		(at 219.71 129.54 0)
+		(effects
+			(font
+				(size 1.27 1.27)
+			)
+			(justify left bottom)
+		)
+	)
 	(label "5V"
 		(at 146.05 54.61 90)
@@
 		)
 	)
+	(label "GPIO_13"
+		(at 204.47 132.08 180)
+		(effects
+			(font
+				(size 1.27 1.27)
+			)
+			(justify right bottom)
+		)
+	)
 	(label "GPIO_7"
 		(at 121.92 88.9 180)
@@
 		)
 	)
-	(label "GPIO_9"
-		(at 204.47 124.46 180)
-		(effects
-			(font
-				(size 1.27 1.27)
-			)
-			(justify right bottom)
-		)
-	)
+	(label "GPIO_12"
+		(at 219.71 132.08 0)
+		(effects
+			(font
+				(size 1.27 1.27)
+			)
+			(justify left bottom)
+		)
+	)
