File: MoBaSbS-502-MoBaStromverteiler/MoBaSbS-502-MoBaStromverteiler.kicad_pcb (KiCad board)
At the start: 2 copper layers, 58.4 x 39.4 mm, 21 parts, among them P1 PSS254, P2 PSS254, P3 PSS254, P4 PSS254, P5 Wago, P6 Wago, P7 PSS254

Commit message: Generated panels, added some new PCBs
Routing:
- net GND: track 165.9 -> 173.5 mm
- net /12V PRE: vias 0 -> 3
- added copper zone on B.Cu, net GND
- added copper zone on F.Cu, net GND
Other:
- board text added: "MoBaSbS-502/1 10.25 Jomer.dev"
- board text removed: "MoBaSbS-502/1"
Changed lines of the file:
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@@
 			(psa4output no)
 			(plot_black_and_white yes)
-			(plotinvisibletext no)
 			(sketchpadsonfab no)
 			(plotpadnumbers no)
@@
 			(layer "F.Fab")
 		)
-		(fp_text user "${REFERENCE}"
-			(at 0 0 180)
-			(layer "F.Fab")
-			(hide yes)
-			(effects
-				(font
-					(size 0.8 0.8)
-					(thickness 0.12)
-				)
-			)
-		)
 		(pad "1" smd roundrect
 			(at -1.4625 0 180)
@@
 			(layer "F.Fab")
 		)
-		(fp_text user "${REFERENCE}"
-			(at 0 0 0)
-			(layer "F.Fab")
-			(hide yes)
-			(effects
-				(font
-					(size 0.8 0.8)
-					(thickness 0.12)
-				)
-			)
-		)
 		(pad "1" smd roundrect
 			(at -1.4625 0)
@@
 			(at 2.54 -4.12 90)
 			(layer "F.SilkS")
+			(hide yes)
 			(effects
 				(font
@@
 			(at 7.62 0 180)
 			(layer "F.SilkS")
+			(hide yes)
 			(effects
 				(font
@@
 			(layer "F.Fab")
 		)
-		(fp_text user "${REFERENCE}"
-			(at 2.54 -2.22 90)
-			(layer "F.Fab")
-			(hide yes)
-			(effects
-				(font
-					(size 1 1)
-					(thickness 0.15)
-				)
-			)
-		)
 		(pad "1" thru_hole roundrect
 			(at 0 0 90)
@@
 			(unlocked yes)
 			(layer "F.SilkS")
+			(hide yes)
 			(effects
 				(font
@@
 			(unlocked yes)
 			(layer "F.SilkS")
+			(hide yes)
 			(effects
 				(font
@@
 			(layer "F.Fab")
 		)
-		(fp_text user "${REFERENCE}"
-			(at 2.5 0 0)
-			(layer "F.Fab")
-			(hide yes)
-			(effects
-				(font
-					(size 1 1)
-					(thickness 0.15)
-				)
-			)
-		)
 		(pad "1" thru_hole rect
 			(at 0 0)
@@
 			(layer "F.Fab")
 		)
-		(fp_text user "${REFERENCE}"
-			(at 2.5 0 0)
-			(layer "F.Fab")
-			(hide yes)
-			(effects
-				(font
-					(size 1 1)
-					(thickness 0.15)
-				)
-			)
-		)
 		(pad "1" thru_hole rect
 			(at 0 0)
@@
 			(layer "F.CrtYd")
 		)
-		(fp_text user "${REFERENCE}"
-			(at 0 0 0)
-			(layer "F.Fab")
-			(hide yes)
-			(effects
-				(font
-					(size 1 1)
-					(thickness 0.15)
-				)
-			)
-		)
 		(pad "1" thru_hole circle
 			(at 0 0)
@@
 			(at 2.54 -4.12 90)
 			(layer "F.SilkS")
+			(hide yes)
 			(effects
 				(font
@@
 			(at 2.54 -4.12 90)
 			(layer "F.SilkS")
+			(hide yes)
 			(effects
 				(font
@@
 			(layer "F.CrtYd")
 		)
-		(fp_text user "${REFERENCE}"
-			(at 0 0 0)
-			(layer "F.Fab")
-			(hide yes)
-			(effects
-				(font
-					(size 1 1)
-					(thickness 0.15)
-				)
-			)
-		)
 		(pad "1" thru_hole circle
 			(at 0 0)
@@
 			(layer "F.CrtYd")
 		)
-		(fp_text user "${REFERENCE}"
-			(at 0 0 0)
-			(layer "F.Fab")
-			(hide yes)
-			(effects
-				(font
-					(size 1 1)
-					(thickness 0.15)
-				)
-			)
-		)
 		(pad "1" thru_hole circle
 			(at 0 0)
@@
 			(layer "F.CrtYd")
 		)
-		(fp_text user "${REFERENCE}"
-			(at 0 0 0)
-			(layer "F.Fab")
-			(hide yes)
-			(effects
-				(font
-					(size 1 1)
-					(thickness 0.15)
-				)
-			)
-		)
 		(pad "1" thru_hole circle
 			(at 0 0)
@@
 			(at 2.54 -4.12 90)
 			(layer "F.SilkS")
+			(hide yes)
 			(effects
 				(font
@@
 			(at 0 1.85 0)
 			(layer "B.SilkS")
+			(hide yes)
 			(effects
 				(font
@@
 			(layer "B.Fab")
 		)
-		(fp_text user "${REFERENCE}"
-			(at 0 0 0)
-			(layer "B.Fab")
-			(hide yes)
-			(effects
-				(font
-					(size 0.8 0.8)
-					(thickness 0.12)
-				)
-				(justify mirror)
-			)
-		)
 		(pad "1" smd roundrect
 			(at -1.475 0)
@@
 			(at 0 1.85 0)
 			(layer "B.SilkS")
+			(hide yes)
 			(effects
 				(font
@@
 			(layer "B.Fab")
 		)
-		(fp_text user "${REFERENCE}"
-			(at 0 0 0)
-			(layer "B.Fab")
-			(hide yes)
-			(effects
-				(font
-					(size 0.8 0.8)
-					(thickness 0.12)
-				)
-				(justify mirror)
-			)
-		)
 		(pad "1" smd roundrect
 			(at -1.475 0)
@@
 		)
 	)
-	(gr_text "MoBaSbS-502/1"
+	(gr_text "MoBaSbS-502/1\n10.25 Jomer.dev"
 		(at 134.84 144.78 0)
 		(layer "F.SilkS")
@@
 	)
 	(segment
-		(start 150.137349 138.372651)
-		(end 150.08 138.43)
-		(width 1)
+		(start 143.857 138.43)
+		(end 147.667 138.43)
+		(width 2)
 		(layer "B.Cu")
 		(net 1)
@@
 	)
 	(segment
-		(start 150.08 138.43)
+		(start 147.667 138.43)
 		(end 131.665 138.43)
 		(width 4)
@@
 	)
 	(segment
+		(start 150.08 138.43)
+		(end 147.667 138.43)
+		(width 4)
+		(layer "B.Cu")
+		(net 1)
+	)
+	(segment
 		(start 158.335 140.335)
 		(end 156.43 138.43)
@@
 	)
 	(segment
+		(start 143.857 134.689651)
+		(end 143.857 138.43)
+		(width 2)
+		(layer "B.Cu")
+		(net 1)
+	)
+	(segment
 		(start 131.722349 138.372651)
 		(end 131.665 138.43)
@@
 	)
 	(segment
+		(start 143.787349 134.62)
+		(end 143.857 134.689651)
+		(width 2)
+		(layer "B.Cu")
+		(net 1)
+	)
+	(segment
 		(start 158.335 136.135001)
 		(end 158.335 140.335)
@@
 	)
 	(segment
+		(start 141.444 153.67)
+		(end 140.682 153.67)
+		(width 1)
+		(layer "B.Cu")
+		(net 4)
+	)
+	(segment
+		(start 140.682 153.67)
+		(end 139.91 153.67)
+		(width 1)
+		(layer "B.Cu")
+		(net 4)
+	)
+	(segment
 		(start 150.5225 152.4)
 		(end 149.2525 153.67)
@@
 	(segment
 		(start 149.2525 153.67)
-		(end 139.91 153.67)
+		(end 141.444 153.67)
 		(width 1)
 		(layer "B.Cu")
@@
 		(net 10)
 	)
+	(via
+		(at 134.205 153.67)
+		(size 0.7)
+		(drill 0.5)
+		(layers "F.Cu" "B.Cu")
+		(net 11)
+	)
+	(via
+		(at 134.205 152.146)
+		(size 0.7)
+		(drill 0.5)
+		(layers "F.Cu" "B.Cu")
+		(net 11)
+	)
+	(via
+		(at 134.205 152.908)
+		(size 0.7)
+		(drill 0.5)
+		(layers "F.Cu" "B.Cu")
+		(net 11)
+	)
 	(segment
 		(start 158.335 146.05)
@@
 	(segment
 		(start 134.205 145.898397)
-		(end 134.205 153.67)
+		(end 134.205 152.146)
 		(width 2)
 		(layer "B.Cu")
@@
 	)
 	(segment
+		(start 134.205 152.908)
+		(end 134.205 153.67)
+		(width 2)
+		(layer "B.Cu")
+		(net 11)
+	)
+	(segment
 		(start 148.658397 144.628397)
 		(end 132.935 144.628397)
@@
 	)
 	(segment
+		(start 134.205 152.146)
+		(end 134.205 152.908)
+		(width 2)
+		(layer "B.Cu")
+		(net 11)
+	)
+	(segment
 		(start 156.324998 148.060002)
 		(end 152.090002 148.060002)
@@
 		(net 11)
 	)
+	(zone
+		(net 1)
+		(net_name "GND")
+		(layers "F.Cu" "B.Cu")
+		(hatch edge 0.5)
+		(connect_pads
+			(clearance 0.508)
+		)
+		(min_thickness 0.25)
+		(filled_areas_thickness no)
+		(fill yes
+			(thermal_gap 0.5)
+			(thermal_bridge_width 0.5)
+			(island_removal_mode 2)
+			(island_area_min 10)
+		)
+		(polygon
+			(pts
+				(xy 107.916 118.11) (xy 166.336 118.11) (xy 166.336 157.48) (xy 107.916 157.48)
+			)
+		)
+	)
 	(embedded_fonts no)
