File: MoBaSbS-505-10Zu4x4/MoBaSbS-505-10Zu4x4.kicad_pcb (KiCad board)
At the start: 2 copper layers, 57.8 x 21.6 mm, 7 parts, among them J1 Conn_02x05_Odd_Even, J10 1, J11 2, J12 3, J13 4

Commit message: Generated panels, added some new PCBs
Other:
- board text added: "1"
- board text added: "2"
- board text added: "3"
- board text added: "4"
- board text added: "MoBaSbS-505/1 10.25 Jomer.dev"
Changed lines of the file:
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@@
 		(layer "Edge.Cuts")
+	)
+	(gr_text "MoBaSbS-505/1\n10.25 Jomer.dev"
+		(at 113.03 96.774 0)
+		(layer "F.SilkS")
+		(effects
+			(font
+				(size 1.5 1.5)
+				(thickness 0.3)
+			)
+		)
+	)
+	(gr_text "4"
+		(at 135.89 82.296 90)
+		(layer "F.SilkS")
+		(effects
+			(font
+				(size 1.5 1.5)
+				(thickness 0.3)
+				(bold yes)
+			)
+		)
+	)
+	(gr_text "3"
+		(at 127 82.423 90)
+		(layer "F.SilkS")
+		(effects
+			(font
+				(size 1.5 1.5)
+				(thickness 0.3)
+				(bold yes)
+			)
+		)
+	)
+	(gr_text "1"
+		(at 109.2 82.423 90)
+		(layer "F.SilkS")
+		(effects
+			(font
+				(size 1.5 1.5)
+				(thickness 0.3)
+				(bold yes)
+			)
+		)
+	)
+	(gr_text "2"
+		(at 118.11 82.423 90)
+		(layer "F.SilkS")
+		(effects
+			(font
+				(size 1.5 1.5)
+				(thickness 0.3)
+				(bold yes)
+			)
+		)
 	)
 	(segment
