File: MA-007-Power/MA-007-Power.kicad_sch (KiCad schematic)
At the start: 14 parts, among them J1 Conn_01x02, J2 Conn_01x03, J3 Power Out

Commit message: Finished up PCBs, added stencil
Parts:
- added J4: 43242-0005, Molex_MiniFitJr_1x3:Molex_MiniFitJr_1x3_PCB, symbol Molex_MiniFitJr1x3_PCB:43242-0005
Connections:
- net 3V3: now also J4.2
- net 5V: now also J4.3; no longer J2.1 (Pin_1)
- net 5V_PRE: now also J2.1 (Pin_1)
- net GND: now also J4.1
Changed lines of the file:
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@@
+	(wire
+		(pts
+			(xy 177.8 111.76) (xy 179.07 111.76)
+		)
+		(stroke
+			(width 0)
+			(type default)
+		)
+	)
 	(wire
 		(pts
@@
 	(wire
 		(pts
+			(xy 177.8 106.68) (xy 179.07 106.68)
+		)
+		(stroke
+			(width 0)
+			(type default)
+		)
+	)
+	(wire
+		(pts
 			(xy 133.35 102.87) (xy 133.35 100.33)
 		)
@@
 	(wire
 		(pts
+			(xy 177.8 109.22) (xy 179.07 109.22)
+		)
+		(stroke
+			(width 0)
+			(type default)
+		)
+	)
+	(wire
+		(pts
 			(xy 130.81 76.2) (xy 138.43 76.2)
 		)
@@
 	)
 	(label "5V"
-		(at 165.1 59.69 180)
+		(at 177.8 106.68 180)
 		(effects
 			(font
@@
 	)
 	(label "GND"
+		(at 177.8 111.76 180)
+		(effects
+			(font
+				(size 1.27 1.27)
+			)
+			(justify right bottom)
+		)
+	)
+	(label "3V3"
+		(at 177.8 109.22 180)
+		(effects
+			(font
+				(size 1.27 1.27)
+			)
+			(justify right bottom)
+		)
+	)
+	(label "GND"
 		(at 130.81 92.71 0)
 		(effects
@@
 	(label "3V3"
 		(at 121.92 100.33 180)
+		(effects
+			(font
+				(size 1.27 1.27)
+			)
+			(justify right bottom)
+		)
+	)
+	(label "5V_PRE"
+		(at 165.1 59.69 180)
 		(effects
 			(font
@@
 					(unit 1)
 				)
+			)
+		)
+	)
+	(symbol
+		(lib_id "Molex_MiniFitJr1x3_PCB:43242-0005")
+		(at 179.07 106.68 0)
+		(unit 1)
+		(exclude_from_sim no)
+		(in_bom yes)
+		(on_board yes)
+		(dnp no)
+		(fields_autoplaced yes)
+		(property "Reference" "J4"
+			(at 195.58 107.9499 0)
+			(effects
+				(font
+					(size 1.27 1.27)
+				)
+				(justify left)
+			)
+		)
+		(property "Value" "43242-0005"
+			(at 195.58 110.4899 0)
+			(effects
+				(font
+					(size 1.27 1.27)
+				)
+				(justify left)
+			)
+		)
+		(property "Footprint" "Molex_MiniFitJr_1x3:Molex_MiniFitJr_1x3_PCB"
+			(at 195.58 201.6 0)
+			(effects
+				(font
+					(size 1.27 1.27)
+				)
+				(justify left top)
+				(hide yes)
+			)
+		)
+		(property "Datasheet" "https://www.molex.com/pdm_docs/sd/432420005_sd.pdf"
+			(at 195.58 301.6 0)
+			(effects
+				(font
+					(size 1.27 1.27)
+				)
+				(justify left top)
+				(hide yes)
+			)
+		)
+		(property "Description" "Headers & Wire Housings MiniFit Jr Header 3 Ckt"
+			(at 179.07 106.68 0)
+			(effects
+				(font
+					(size 1.27 1.27)
+				)
+				(hide yes)
+			)
+		)
+		(property "Height" "12.83"
+			(at 195.58 501.6 0)
+			(effects
+				(font
+					(size 1.27 1.27)
+				)
+				(justify left top)
+				(hide yes)
+			)
+		)
+		(property "Mouser Part Number" "538-43242-0005"
+			(at 195.58 601.6 0)
+			(effects
+				(font
+					(size 1.27 1.27)
+				)
+				(justify left top)
+				(hide yes)
+			)
+		)
+		(property "Mouser Price/Stock" "https://www.mouser.co.uk/ProductDetail/Molex/43242-0005?qs=WXzVXFlun0UzpNSBTvE%252BTg%3D%3D"
+			(at 195.58 701.6 0)
+			(effects
+				(font
+					(size 1.27 1.27)
+				)
+				(justify left top)
+				(hide yes)
+			)
+		)
+		(property "Manufacturer_Name" "Molex"
+			(at 195.58 801.6 0)
+			(effects
+				(font
+					(size 1.27 1.27)
+				)
+				(justify left top)
+				(hide yes)
+			)
+		)
+		(property "Manufacturer_Part_Number" "43242-0005"
+			(at 195.58 901.6 0)
+			(effects
+				(font
+					(size 1.27 1.27)
+				)
+				(justify left top)
+				(hide yes)
+			)
+		)
+		(pin "3"
+		)
+		(pin "1"
+		)
+		(pin "2"
+		)
+		(instances
+			(project "MA-007-Power"
+				(path "/d43a0742-6de7-4807-8d17-3401e22deab4"
+					(reference "J4")
+					(unit 1)
+				)
