File: MoBaSbS-503-BoosterStromSplitter/MoBaSbS-503-BoosterStromSplitter.kicad_pcb (KiCad board)
At the start: 2 copper layers, 12.7 x 64.5 mm, 5 parts, among them J1 39-28-1043, J2 39-28-1043, J3 39-28-1043, J4 39-28-1043, J5 39-28-1043

Commit message: Finished up PCBs, added stencil
Parts:
- added H1: MountingHole_Pad, MountingHole:MountingHole_2.7mm_M2.5_DIN965_Pad, F.Cu at (137.9, 37.7)
- added H3: MountingHole_Pad, MountingHole:MountingHole_2.7mm_M2.5_DIN965_Pad, F.Cu at (137.9, 108.7)
Other:
- board size 12.7 x 64.5 mm -> 12.7 x 77 mm
- board text added: "MoBaSbs-503/1 10.25 Jomer.dev"
Changed lines of the file:
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@@
 			(psa4output no)
 			(plot_black_and_white yes)
-			(plotinvisibletext no)
 			(sketchpadsonfab no)
 			(plotpadnumbers no)
@@
 	(net 11 "/GND")
 	(net 12 "/POW")
+	(net 13 "unconnected-(H1-Pad1)")
+	(net 14 "unconnected-(H3-Pad1)")
+	(footprint "MountingHole:MountingHole_2.7mm_M2.5_DIN965_Pad"
+		(layer "F.Cu")
+		(at 137.922 37.719)
+		(descr "Mounting Hole 2.7mm, M2.5, DIN965")
+		(tags "mounting hole 2.7mm m2.5 din965")
+		(property "Reference" "H1"
+			(at 0 -3.35 0)
+			(layer "F.SilkS")
+			(hide yes)
+			(effects
+				(font
+					(size 1 1)
+					(thickness 0.15)
+				)
+			)
+		)
+		(property "Value" "MountingHole_Pad"
+			(at 0 3.35 0)
+			(layer "F.Fab")
+			(effects
+				(font
+					(size 1 1)
+					(thickness 0.15)
+				)
+			)
+		)
+		(property "Datasheet" "~"
+			(at 0 0 0)
+			(unlocked yes)
+			(layer "F.Fab")
+			(hide yes)
+			(effects
+				(font
+					(size 1.27 1.27)
+					(thickness 0.15)
+				)
+			)
+		)
+		(property "Description" ""
+			(at 0 0 0)
+			(unlocked yes)
+			(layer "F.Fab")
+			(hide yes)
+			(effects
+				(font
+					(size 1.27 1.27)
+					(thickness 0.15)
+				)
+			)
+		)
+		(property ki_fp_filters "MountingHole*Pad*")
+		(sheetname "/")
+		(sheetfile "MoBaSbS-503-BoosterStromSplitter.kicad_sch")
+		(attr exclude_from_pos_files)
+		(fp_circle
+			(center 0 0)
+			(end 2.35 0)
+			(stroke
+				(width 0.15)
+				(type solid)
+			)
+			(fill no)
+			(layer "Cmts.User")
+		)
+		(fp_circle
+			(center 0 0)
+			(end 2.6 0)
+			(stroke
+				(width 0.05)
+				(type solid)
+			)
+			(fill no)
+			(layer "F.CrtYd")
+		)
+		(fp_text user "${REFERENCE}"
+			(at 0 0 0)
+			(layer "F.Fab")
+			(effects
+				(font
+					(size 1 1)
+					(thickness 0.15)
+				)
+			)
+		)
+		(pad "1" thru_hole circle
+			(at 0 0)
+			(size 4.7 4.7)
+			(drill 2.7)
+			(layers "*.Cu" "*.Mask")
+			(remove_unused_layers no)
+			(net 13 "unconnected-(H1-Pad1)")
+			(pinfunction "1")
+			(pintype "input+no_connect")
+		)
+		(embedded_fonts no)
+	)
 	(footprint "Molex_MiniFitJr_2x2_PCB:Molex_MiniFitJr_2x2_PCB"
 		(layer "F.Cu")
@@
 			)
 			(layer "F.Fab")
-		)
-		(fp_text user "${REFERENCE}"
-			(at 0 0 90)
-			(layer "F.Fab")
-			(hide yes)
-			(effects
-				(font
-					(size 1.27 1.27)
-					(thickness 0.254)
-				)
-			)
 		)
 		(pad "1" thru_hole rect
@@
 			(layer "F.Fab")
 		)
-		(fp_text user "${REFERENCE}"
-			(at 0 0 90)
-			(layer "F.Fab")
-			(hide yes)
-			(effects
-				(font
-					(size 1.27 1.27)
-					(thickness 0.254)
-				)
-			)
-		)
 		(pad "1" thru_hole rect
 			(at 0 0 90)
@@
 		)
 	)
+	(footprint "MountingHole:MountingHole_2.7mm_M2.5_DIN965_Pad"
+		(layer "F.Cu")
+		(at 137.922 108.712)
+		(descr "Mounting Hole 2.7mm, M2.5, DIN965")
+		(tags "mounting hole 2.7mm m2.5 din965")
+		(property "Reference" "H3"
+			(at 0 -3.35 0)
+			(layer "F.SilkS")
+			(hide yes)
+			(effects
+				(font
+					(size 1 1)
+					(thickness 0.15)
+				)
+			)
+		)
+		(property "Value" "MountingHole_Pad"
+			(at 0 3.35 0)
+			(layer "F.Fab")
+			(effects
+				(font
+					(size 1 1)
+					(thickness 0.15)
+				)
+			)
+		)
+		(property "Datasheet" "~"
+			(at 0 0 0)
+			(unlocked yes)
+			(layer "F.Fab")
+			(hide yes)
+			(effects
+				(font
+					(size 1.27 1.27)
+					(thickness 0.15)
+				)
+			)
+		)
+		(property "Description" ""
+			(at 0 0 0)
+			(unlocked yes)
+			(layer "F.Fab")
+			(hide yes)
+			(effects
+				(font
+					(size 1.27 1.27)
+					(thickness 0.15)
+				)
+			)
+		)
+		(property ki_fp_filters "MountingHole*Pad*")
+		(sheetname "/")
+		(sheetfile "MoBaSbS-503-BoosterStromSplitter.kicad_sch")
+		(attr exclude_from_pos_files)
+		(fp_circle
+			(center 0 0)
+			(end 2.35 0)
+			(stroke
+				(width 0.15)
+				(type solid)
+			)
+			(fill no)
+			(layer "Cmts.User")
+		)
+		(fp_circle
+			(center 0 0)
+			(end 2.6 0)
+			(stroke
+				(width 0.05)
+				(type solid)
+			)
+			(fill no)
+			(layer "F.CrtYd")
+		)
+		(fp_text user "${REFERENCE}"
+			(at 0 0 0)
+			(layer "F.Fab")
+			(effects
+				(font
+					(size 1 1)
+					(thickness 0.15)
+				)
+			)
+		)
+		(pad "1" thru_hole circle
+			(at 0 0)
+			(size 4.7 4.7)
+			(drill 2.7)
+			(layers "*.Cu" "*.Mask")
+			(remove_unused_layers no)
+			(net 14 "unconnected-(H3-Pad1)")
+			(pinfunction "1")
+			(pintype "input+no_connect")
+		)
+		(embedded_fonts no)
+	)
 	(footprint "Molex_MiniFitJr_2x2_PCB:Molex_MiniFitJr_2x2_PCB"
 		(layer "F.Cu")
@@
 			)
 			(layer "F.Fab")
-		)
-		(fp_text user "${REFERENCE}"
-			(at 0 0 90)
-			(layer "F.Fab")
-			(hide yes)
-			(effects
-				(font
-					(size 1.27 1.27)
-					(thickness 0.254)
-				)
-			)
 		)
 		(pad "1" thru_hole rect
@@
 			(layer "F.Fab")
 		)
-		(fp_text user "${REFERENCE}"
-			(at 0 0 90)
-			(layer "F.Fab")
-			(hide yes)
-			(effects
-				(font
-					(size 1.27 1.27)
-					(thickness 0.254)
-				)
-			)
-		)
 		(pad "1" thru_hole rect
 			(at 0 0 90)
@@
 			(layer "F.Fab")
 		)
-		(fp_text user "${REFERENCE}"
-			(at 0 0 90)
-			(layer "F.Fab")
-			(hide yes)
-			(effects
-				(font
-					(size 1.27 1.27)
-					(thickness 0.254)
-				)
-			)
-		)
 		(pad "1" thru_hole rect
 			(at 0 0 90)
@@
 	)
 	(gr_line
-		(start 144.272 106.172)
-		(end 131.572 106.172)
+		(start 144.272 111.76)
+		(end 131.572 111.76)
 		(stroke
 			(width 0.05)
@@
 	)
 	(gr_line
-		(start 131.572 41.656)
-		(end 144.272 41.656)
+		(start 131.572 34.798)
+		(end 144.272 34.798)
 		(stroke
 			(width 0.05)
@@
 	)
 	(gr_line
-		(start 144.272 41.656)
-		(end 144.272 106.172)
+		(start 144.272 34.798)
+		(end 144.272 111.76)
 		(stroke
 			(width 0.05)
@@
 	)
 	(gr_line
-		(start 131.572 106.172)
-		(end 131.572 41.656)
+		(start 131.572 111.76)
+		(end 131.572 34.798)
 		(stroke
 			(width 0.05)
@@
 		)
 		(layer "Edge.Cuts")
+	)
+	(gr_text "MoBaSbs-503/1 10.25 Jomer.dev"
+		(at 133.731 70.866 90)
+		(layer "B.SilkS")
+		(effects
+			(font
+				(size 1.2 1.2)
+				(thickness 0.3)
+				(bold yes)
+			)
+			(justify bottom mirror)
+		)
 	)
 	(segment
@@
 		(polygon
 			(pts
-				(xy 131.572 41.656) (xy 131.572 106.172) (xy 144.272 106.172) (xy 144.272 41.656)
+				(xy 131.572 34.798) (xy 131.572 111.76) (xy 144.272 111.76) (xy 144.272 34.798)
 			)
 		)
@@
 		(polygon
 			(pts
-				(xy 131.572 41.656) (xy 131.572 106.172) (xy 144.272 106.172) (xy 144.272 41.656)
-			)
-		)
+				(xy 131.572 34.798) (xy 131.572 111.76) (xy 144.272 111.76) (xy 144.272 34.798)
+			)
+		)
