File: MoBaSbS-510-AnschaltGruppev3/MoBaSbS-002-AnschaltGruppev3.kicad_pcb (KiCad board)
At the start: 2 copper layers, 58.4 x 80 mm, 37 parts, among them IC1 TJA1057BT, IC2 SP3485EN-L_TR, IC3 MCP2518FDT-E_SL, J1 RJ45, J2 RJ45, J3 Conn_02x03_Odd_Even, J4 Conn_01x03, J5 Conn_02x05_Counter_Clockwise, J6 Conn_01x04, J7 Conn_01x04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

Commit message: Finished up PCBs, added stencil
Parts:
- added J10: Conn_01x02, Connector_PinHeader_2.54mm:PinHeader_1x02_P2.54mm_Vertical_SMD_Pin1Left, F.Cu at (140.3, 95.5)
- added J9: Conn_01x03, Connector_PinHeader_2.54mm:PinHeader_1x03_P2.54mm_Vertical_SMD_Pin1Left, F.Cu at (140.3, 87.8)
- D3: footprint LED_SMD:LED_WS2812B-2020_PLCC4_2.0x2.0mm -> LED_SMD:LED_WS2812B-Mini_PLCC4_3.5x3.5mm
- IC3: footprint CAN Controller:SOIC127P600X175-14N -> SOIC127P600X175-14N:SOIC127P600X175-14N
Connections:
- A1 pad 36: /+3V3 -> /+3V3_PICO
- A1 pad 39: unconnected-(A1-VSYS-Pad39) -> +5V
- A1 pad 40: +5V -> unconnected-(A1-VBUS-Pad40)
- IC1 pad 8: unconnected-(IC1-S-Pad8) -> /+3V3
Routing:
- net GND: track 201.3 -> 222.5 mm
- net /+3V3: track 54.4 -> 62.5 mm, vias 3 -> 2
- net +5V: track 203.0 -> 208.4 mm, vias 3 -> 6
- net /+3V3_PICO: track 0.00 -> 4.44 mm, vias 0 -> 1
- net /WS2812: track 43.8 -> 42.9 mm
Other:
- board text added: "3V3 external"
- board text added: "3V3 from Pico"
- board text added: "MoBaSbS-510/1 10.25 Jomer.dev"
- board text removed: "J1"
- board text removed: "J2"
- board text removed: "MoBaSbS 002/3"
- board text removed: "MoBaSbS-002/3"
