File: MoBaSbS-511-GPIO/MoBaSbS-511-GPIO.kicad_sch (KiCad schematic)
At the start: 36 parts, among them J1 Conn_02x05_Counter_Clockwise, J2 Conn_02x06_Odd_Even, J5 Conn_02x05_Counter_Clockwise, P1 2x5_Buchse, P3 PSS-3G, P4 PSS-3G, P5 2x5_Buchse, U1 PCA9685PW

Commit message: Finished up PCBs, added stencil
Parts:
- removed J2: Conn_02x06_Odd_Even, Connector_PinHeader_2.54mm:PinHeader_2x06_P2.54mm_Vertical, symbol Connector_Generic:Conn_02x06_Odd_Even
- removed R10, R11, R12, R13, R14, R20, R21, R22, R23, R24, R25, R26, R27, R7, R8, R9: R, Resistor_SMD:R_1206_3216Metric_Pad1.30x1.75mm_HandSolder, symbol MoBaSbS-004-1-AtMega8-rescue:R
- removed R4, R5, R6: R, Resistor_SMD:R_0603_1608Metric_Pad0.98x0.95mm_HandSolder, symbol MoBaSbS-004-1-AtMega8-rescue:R
- removed U1: PCA9685PW, Package_SO:TSSOP-28_4.4x9.7mm_P0.65mm, symbol Driver_LED:PCA9685PW
- added J2: Conn_02x03_Odd_Even, Connector_PinHeader_2.54mm:PinHeader_2x03_P2.54mm_Vertical, symbol Connector_Generic:Conn_02x03_Odd_Even
- added U1: MCP23017_SS, Package_SO:SSOP-28_5.3x10.2mm_P0.65mm, symbol Interface_Expansion:MCP23017_SS
Connections:
- net +5V: now also J2.1 (Pin_1), J2.3 (Pin_3), J2.5 (Pin_5), U1.18 (~{RESET}), U1.9 (VDD)
- net GND: now also U1.10 (VSS)
- net I2C_SCL: now also U1.12 (SCK)
- net I2C_SDA: now also U1.13 (SDA)
- net at R1.2: now also J2.2 (Pin_2), U1.15 (A0)
- net at R3.2: now also J2.6 (Pin_6), U1.17 (A2)
- net at R2.2: now also J2.4 (Pin_4), U1.16 (A1)
- net LED_0 renamed GPIO_0
- net GPIO_0: now also U1.28 (GPA7)
- net LED_1 renamed GPIO_1
- net GPIO_1: now also U1.27 (GPA6)
- net LED_10 renamed GPIO_10
- net GPIO_10: now also U1.6 (GPB5)
- net LED_11 renamed GPIO_11
- net GPIO_11: now also U1.5 (GPB4)
- net LED_12 renamed GPIO_12
- net GPIO_12: now also U1.4 (GPB3)
- net LED_13 renamed GPIO_13
- net GPIO_13: now also U1.3 (GPB2)
- net LED_14 renamed GPIO_14
- net GPIO_14: now also U1.2 (GPB1)
- net LED_15 renamed GPIO_15
- net GPIO_15: now also U1.1 (GPB0)
- net LED_2 renamed GPIO_2
- net GPIO_2: now also U1.26 (GPA5)
- net LED_3 renamed GPIO_3
- net GPIO_3: now also U1.25 (GPA4)
- net LED_4 renamed GPIO_4
- net GPIO_4: now also U1.24 (GPA3)
- net LED_5 renamed GPIO_5
- net GPIO_5: now also U1.23 (GPA2)
- net LED_6 renamed GPIO_6
- net GPIO_6: now also U1.22 (GPA1)
- net LED_7 renamed GPIO_7
- net GPIO_7: now also U1.21 (GPA0)
- net LED_8 renamed GPIO_8
- net GPIO_8: now also U1.8 (GPB7)
- net LED_9 renamed GPIO_9
- net GPIO_9: now also U1.7 (GPB6)
- no-connect marks 4 -> 5
Other:
- moved on the sheet: R1, R2, R3
