File: MoBaSbS-511-GPIO/MoBaSbS-511-GPIO.kicad_pcb (KiCad board)
At the start: 2 copper layers, 36.2 x 81.3 mm, 17 parts, among them J1 Conn_02x05_Counter_Clockwise, J2 Conn_02x03_Odd_Even, J5 Conn_02x05_Counter_Clockwise, P1 2x5_Buchse, P3 PSS-3G, P4 PSS-3G, P5 2x5_Buchse, U1 MCP23017_SS

Commit message: Latest changes
Changed lines of the file:
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@@
 			(at 1.27 -6.1 0)
 			(layer "F.SilkS")
+			(hide yes)
 			(effects
 				(font
@@
 			(at -5.65 -2.77 0)
 			(layer "F.SilkS")
+			(hide yes)
 			(effects
 				(font
@@
 			(at 0 -1.43 90)
 			(layer "F.SilkS")
+			(hide yes)
 			(effects
 				(font
@@
 			(at 5.655 -2.27 0)
 			(layer "F.SilkS")
+			(hide yes)
 			(effects
 				(font
