File: Stencil/Stencil.kicad_pcb (KiCad board)
At the start: 2 copper layers, 150 x 150 mm, 60 parts, among them IC1 TJA1057BT, IC2 SP3485EN-L_TR, IC3 MCP2518FDT-E_SL, J10 Conn_01x02, J9 Conn_01x03, U1 MCP23017_SS, U1 PCA9685PW

Commit message: Latest changes
Parts:
- added C1: 100nF, Capacitors_SMD:C_1206, F.Cu at (64.8, 126.4)
- added C1: 100nF, Capacitors_SMD:C_1206, F.Cu at (64.8, 145.4)
- added C1: 100nF, Capacitors_SMD:C_1206, F.Cu at (64.8, 158.1)
- added C1: 100nF, Capacitors_SMD:C_1206, F.Cu at (64.8, 107.3)
- added C1: 100nF, Capacitors_SMD:C_1206, F.Cu at (64.8, 120.0)
- added C1: 100nF, Capacitors_SMD:C_1206, F.Cu at (64.8, 132.7)
- added C1: 100nF, Capacitors_SMD:C_1206, F.Cu at (64.8, 113.7)
- added C1: 100nF, Capacitors_SMD:C_1206, F.Cu at (64.8, 151.8)
- added C1: 100nF, Capacitors_SMD:C_1206, F.Cu at (64.8, 139.1)
- added C1: 100nF, Capacitors_SMD:C_1206, F.Cu at (64.8, 101.0)
- added C2: 10nF, Capacitors_SMD:C_1206, F.Cu at (67.3, 151.8)
- added C2: 10nF, Capacitors_SMD:C_1206, F.Cu at (67.3, 139.1)
- added C2: 10nF, Capacitors_SMD:C_1206, F.Cu at (67.3, 158.1)
- added C2: 10nF, Capacitors_SMD:C_1206, F.Cu at (67.3, 120.0)
- added C2: 10nF, Capacitors_SMD:C_1206, F.Cu at (67.3, 132.7)
- added C2: 10nF, Capacitors_SMD:C_1206, F.Cu at (67.3, 101.0)
- added C2: 10nF, Capacitors_SMD:C_1206, F.Cu at (67.3, 113.7)
- added C2: 10nF, Capacitors_SMD:C_1206, F.Cu at (67.3, 145.4)
- added C2: 10nF, Capacitors_SMD:C_1206, F.Cu at (67.3, 107.3)
- added C2: 10nF, Capacitors_SMD:C_1206, F.Cu at (67.3, 126.4)
Other:
- board text added: "MoBaSbS-058"
